Commit message: Publish MMC dynamics, controllers and reproducible simulation experiments

File: src/mmc_uav_description/urdf/mmc_uav.urdf (robot description, URDF)
Before this commit: robot mmc_uav_description, 7 links, 6 joints
Joints:
- joint joint_rotor_lower: origin xyz=0 0 0.02 rpy=0 0 0 -> xyz=1.2765511418678223e-10 -9.3711794139119825e-06 -0.014763627586206887 rpy=0 0 0
- joint joint_rotor_upper: origin xyz=0 0 0.05 rpy=0 0 0 -> xyz=1.2765511418678223e-10 -9.3711794139119825e-06 0.015236372413793116 rpy=0 0 0
- joint joint_slider_blue: origin xyz=0.18 0.00015028 0.0050303 rpy=0 0 0 -> xyz=0.1800000001276551 0.00014090882058608801 -0.029733327586206885 rpy=0 0 0
- joint joint_slider_green: origin xyz=0 0.18 0.0050303 rpy=0 0 0 -> xyz=1.2765511418678223e-10 0.17999062882058608 -0.029733327586206885 rpy=0 0 0
- joint joint_slider_purple: origin xyz=0 -0.18 0.0050303 rpy=0 0 0 -> xyz=1.2765511418678223e-10 -0.1800093711794139 -0.029733327586206885 rpy=0 0 0
- joint joint_slider_red: origin xyz=-0.18 0.00012143 0.0050303 rpy=0 0 0 -> xyz=-0.17999999987234488 0.00011205882058608802 -0.029733327586206885 rpy=0 0 0
